File: hardware/eagle/rpi-cc2520-interface/rev_b/interface_b.brd (EAGLE design)
At the start: 30.5 x 39.5 mm, 11 parts, among them J1 PINHD-2X12/SMD, J2 PINHD-2X12/SMD

Commit message: shipped version of the board
Connections:
- net GPIO17 renamed !RESET
Other:
- board text added: "!RST"
- board text added: "2013/02/11"
- board text removed: "2013/02/07"
- board text removed: "G17"
Changed lines of the file:
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@@
 Interface</text>
 <text x="18.669" y="37.846" size="1.016" layer="21" font="vector" ratio="12" align="bottom-center">Brad Campbell</text>
-<text x="22.098" y="19.812" size="1.016" layer="21" font="vector" ratio="12" align="bottom-center">2013/02/07</text>
+<text x="22.098" y="19.812" size="1.016" layer="21" font="vector" ratio="12" align="bottom-center">2013/02/11</text>
 <text x="7.747" y="3.048" size="0.762" layer="21" font="vector" ratio="10" align="center-left">3.3V</text>
 <text x="2.667" y="3.048" size="0.762" layer="21" font="vector" ratio="10" align="center-right">5V</text>
@@
 <text x="7.747" y="10.668" size="0.762" layer="21" font="vector" ratio="10" align="center-left">LED0</text>
 <text x="7.747" y="13.208" size="0.762" layer="21" font="vector" ratio="10" align="center-left">GND</text>
-<text x="7.747" y="15.748" size="0.762" layer="21" font="vector" ratio="10" align="center-left">G17</text>
+<text x="7.747" y="15.748" size="0.762" layer="21" font="vector" ratio="10" align="center-left">!RST</text>
 <text x="7.747" y="18.288" size="0.762" layer="21" font="vector" ratio="10" align="center-left">LED2</text>
 <text x="7.747" y="20.828" size="0.762" layer="21" font="vector" ratio="10" align="center-left">CCA</text>
@@
 <wire x1="3.81" y1="24.638" x2="1.524" y2="24.638" width="0.8128" layer="16"/>
 </signal>
-<signal name="GPIO17">
+<signal name="!RESET">
 <contactref element="J1" pad="12"/>
 <contactref element="J2" pad="11"/>
