File: hardware/eagle/rpi-cc2520-interface/rev_b/interface_b.sch (EAGLE design)
At the start: 11 parts, among them J1 PINHD-2X12/SMD, J2 PINHD-2X12/SMD

Commit message: shipped version of the board
Connections:
- net GPIO17 renamed !RESET
Changed lines of the file:
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@@
 </segment>
 </net>
-<net name="GPIO17" class="0">
+<net name="!RESET" class="0">
 <segment>
 <pinref part="J1" gate="G$1" pin="12"/>
