File: hardware/eagle/rpi-cc2520/rev_a/rpi-cc2520_a.sch (EAGLE design)
At the start: 22 parts, among them P1 MOLEX_73251-135X, U1 CC2520, X1 NX2520SA

Commit message: Added ID chip to board.
This is important for creating a mac address. Otherwise the 15.4 side
doesn't have a good way of getting a unique address.
Parts:
- added R6: 2.2k, rcl:R-US_R0402
- added U2: DS2411, chips:DS2411
- R1, R2, R3: device rcl:R-US_R0603 -> rcl:R-US_R0402; DIGIKEY (none) -> RHM470JCT-ND
Connections:
- removed net UART0_TXD: J1.8
- new net ID_DATA: J1.8, R6.1, U2.I/O
- net GND: now also U2.GND
- net VCC: now also R6.2, U2.VCC
Changed lines of the file:
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@@
 <attribute name="DIGIKEY" value="160-1837-1-ND"/>
 </part>
-<part name="R1" library="rcl" deviceset="R-US_" device="R0603" value="470"/>
-<part name="R2" library="rcl" deviceset="R-US_" device="R0603" value="470"/>
-<part name="R3" library="rcl" deviceset="R-US_" device="R0603" value="470"/>
 <part name="P+1" library="SparkFun" deviceset="VCC" device=""/>
 <part name="P+2" library="SparkFun" deviceset="VCC" device=""/>
@@
 <part name="B1" library="rpi-cc2520" deviceset="2450BM15A0002" device=""/>
 <part name="GND1" library="supply1" deviceset="GND" device=""/>
+<part name="U2" library="chips" deviceset="DS2411" device=""/>
+<part name="GND7" library="supply1" deviceset="GND" device=""/>
+<part name="P+4" library="SparkFun" deviceset="VCC" device=""/>
+<part name="R6" library="rcl" deviceset="R-US_" device="R0402" value="2.2k">
+<attribute name="DIGIKEY" value="RHM2.2KCECT-ND"/>
+</part>
+<part name="P+6" library="SparkFun" deviceset="VCC" device=""/>
+<part name="R1" library="rcl" deviceset="R-US_" device="R0402" value="470">
+<attribute name="DIGIKEY" value="RHM470JCT-ND"/>
+</part>
+<part name="R2" library="rcl" deviceset="R-US_" device="R0402" value="470">
+<attribute name="DIGIKEY" value="RHM470JCT-ND"/>
+</part>
+<part name="R3" library="rcl" deviceset="R-US_" device="R0402" value="470">
+<attribute name="DIGIKEY" value="RHM470JCT-ND"/>
+</part>
 </parts>
 <sheets>
@@
 <attribute name="DIGIKEY" x="233.68" y="96.52" size="1.27" layer="96" display="off"/>
 </instance>
-<instance part="R1" gate="G$1" x="213.36" y="86.36" rot="R90"/>
-<instance part="R2" gate="G$1" x="223.52" y="86.36" rot="R90"/>
-<instance part="R3" gate="G$1" x="233.68" y="86.36" rot="R90"/>
 <instance part="P+1" gate="1" x="213.36" y="101.6"/>
 <instance part="P+2" gate="1" x="223.52" y="101.6"/>
@@
 <instance part="B1" gate="G$1" x="142.24" y="73.66"/>
 <instance part="GND1" gate="1" x="157.48" y="58.42"/>
+<instance part="U2" gate="G$1" x="30.48" y="25.4"/>
+<instance part="GND7" gate="1" x="43.18" y="17.78"/>
+<instance part="P+4" gate="1" x="43.18" y="40.64"/>
+<instance part="R6" gate="G$1" x="50.8" y="33.02" rot="R90">
+<attribute name="DIGIKEY" x="50.8" y="33.02" size="1.27" layer="96" rot="R90" display="off"/>
+</instance>
+<instance part="P+6" gate="1" x="50.8" y="40.64"/>
+<instance part="R1" gate="G$1" x="213.36" y="86.36" rot="R90">
+<attribute name="DIGIKEY" x="213.36" y="86.36" size="1.27" layer="96" rot="R90" display="off"/>
+</instance>
+<instance part="R2" gate="G$1" x="223.52" y="86.36" rot="R90">
+<attribute name="DIGIKEY" x="223.52" y="86.36" size="1.27" layer="96" rot="R90" display="off"/>
+</instance>
+<instance part="R3" gate="G$1" x="233.68" y="86.36" rot="R90">
+<attribute name="DIGIKEY" x="233.68" y="86.36" size="1.27" layer="96" rot="R90" display="off"/>
+</instance>
 </instances>
 <busses>
 </busses>
 <nets>
-<net name="UART0_TXD" class="0">
-<segment>
-<pinref part="J1" gate="A" pin="8"/>
-<wire x1="132.842" y1="166.116" x2="127.762" y2="166.116" width="0.1524" layer="91"/>
-<label x="132.842" y="166.116" size="1.27" layer="95" xref="yes"/>
-</segment>
-</net>
 <net name="UART0_RXD" class="0">
 <segment>
@@
 <pinref part="GND1" gate="1" pin="GND"/>
 </segment>
+<segment>
+<pinref part="U2" gate="G$1" pin="GND"/>
+<wire x1="40.64" y1="22.86" x2="43.18" y2="22.86" width="0.1524" layer="91"/>
+<wire x1="43.18" y1="22.86" x2="43.18" y2="20.32" width="0.1524" layer="91"/>
+<pinref part="GND7" gate="1" pin="GND"/>
+</segment>
 </net>
 <net name="!RESET" class="0">
@@
 </segment>
 </net>
-<net name="N$1" class="0">
-<segment>
-<pinref part="D1" gate="G$1" pin="C"/>
-<pinref part="R1" gate="G$1" pin="2"/>
-</segment>
-</net>
-<net name="N$2" class="0">
-<segment>
-<pinref part="D2" gate="G$1" pin="C"/>
-<pinref part="R2" gate="G$1" pin="2"/>
-</segment>
-</net>
-<net name="N$3" class="0">
-<segment>
-<pinref part="D3" gate="G$1" pin="C"/>
-<pinref part="R3" gate="G$1" pin="2"/>
-</segment>
-</net>
 <net name="VCC" class="0">
 <segment>
@@
 <pinref part="P+5" gate="1" pin="VCC"/>
 </segment>
+<segment>
+<pinref part="U2" gate="G$1" pin="VCC"/>
+<wire x1="40.64" y1="27.94" x2="43.18" y2="27.94" width="0.1524" layer="91"/>
+<wire x1="43.18" y1="27.94" x2="43.18" y2="40.64" width="0.1524" layer="91"/>
+<pinref part="P+4" gate="1" pin="VCC"/>
+</segment>
+<segment>
+<pinref part="P+6" gate="1" pin="VCC"/>
+<pinref part="R6" gate="G$1" pin="2"/>
+<wire x1="50.8" y1="40.64" x2="50.8" y2="38.1" width="0.1524" layer="91"/>
+</segment>
 </net>
 <net name="LED2" class="0">
 <segment>
-<pinref part="R3" gate="G$1" pin="1"/>
 <wire x1="233.68" y1="81.28" x2="233.68" y2="73.66" width="0.1524" layer="91"/>
 <wire x1="233.68" y1="73.66" x2="210.82" y2="73.66" width="0.1524" layer="91"/>
 <label x="210.82" y="73.66" size="1.27" layer="95" rot="R180" xref="yes"/>
+<pinref part="R3" gate="G$1" pin="1"/>
 </segment>
 <segment>
@@
 <net name="LED1" class="0">
 <segment>
-<pinref part="R2" gate="G$1" pin="1"/>
 <wire x1="223.52" y1="81.28" x2="223.52" y2="76.2" width="0.1524" layer="91"/>
 <wire x1="223.52" y1="76.2" x2="210.82" y2="76.2" width="0.1524" layer="91"/>
 <label x="210.82" y="76.2" size="1.27" layer="95" rot="R180" xref="yes"/>
+<pinref part="R2" gate="G$1" pin="1"/>
 </segment>
 <segment>
@@
 <net name="LED0" class="0">
 <segment>
-<pinref part="R1" gate="G$1" pin="1"/>
 <wire x1="213.36" y1="81.28" x2="213.36" y2="78.74" width="0.1524" layer="91"/>
 <wire x1="213.36" y1="78.74" x2="210.82" y2="78.74" width="0.1524" layer="91"/>
 <label x="210.82" y="78.74" size="1.27" layer="95" rot="R180" xref="yes"/>
+<pinref part="R1" gate="G$1" pin="1"/>
 </segment>
 <segment>
@@
 </segment>
 </net>
+<net name="ID_DATA" class="0">
+<segment>
+<pinref part="U2" gate="G$1" pin="I/O"/>
+<wire x1="40.64" y1="25.4" x2="50.8" y2="25.4" width="0.1524" layer="91"/>
+<label x="55.88" y="25.4" size="1.27" layer="95" xref="yes"/>
+<pinref part="R6" gate="G$1" pin="1"/>
+<wire x1="50.8" y1="25.4" x2="55.88" y2="25.4" width="0.1524" layer="91"/>
+<wire x1="50.8" y1="27.94" x2="50.8" y2="25.4" width="0.1524" layer="91"/>
+<junction x="50.8" y="25.4"/>
+</segment>
+<segment>
+<pinref part="J1" gate="A" pin="8"/>
+<wire x1="132.842" y1="166.116" x2="127.762" y2="166.116" width="0.1524" layer="91"/>
+<label x="132.842" y="166.116" size="1.27" layer="95" xref="yes"/>
+</segment>
+</net>
+<net name="N$1" class="0">
+<segment>
+<pinref part="D1" gate="G$1" pin="C"/>
+<pinref part="R1" gate="G$1" pin="2"/>
+</segment>
+</net>
+<net name="N$2" class="0">
+<segment>
+<pinref part="D2" gate="G$1" pin="C"/>
+<pinref part="R2" gate="G$1" pin="2"/>
+</segment>
+</net>
+<net name="N$3" class="0">
+<segment>
+<pinref part="D3" gate="G$1" pin="C"/>
+<pinref part="R3" gate="G$1" pin="2"/>
+</segment>
+</net>
